File: TeensyDSP_Hardware.kicad_sch (KiCad schematic)
At the start: 57 parts, among them J1 AudioJack2, J2 AudioJack2, J3 Conn_01x04_Pin, SW2 SW_DPDT_x2, SW3 SW_SPDT, U1 TL071, U2 LTC1044, U3 TL071, U4 TL071, U5 TL071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

Commit message: final commit before change to single ended
Parts:
- removed C10, C11, C12, C13, C14, C7, C8, C9: C, Capacitor_THT:C_Disc_D4.3mm_W1.9mm_P5.00mm, symbol Device:C
- removed J2: AudioJack2, Connector_Audio:Jack_3.5mm_Ledino_KB3SPRS_Horizontal, symbol Connector_Audio:AudioJack2
- removed R13, R14, R15, R16, R17, R18, R19: R, Resistor_THT:R_Axial_DIN0207_L6.3mm_D2.5mm_P7.62mm_Horizontal, symbol Device:R
- removed U4, U5: TL071, Package_DIP:DIP-8_W7.62mm, symbol Amplifier_Operational:TL071
- removed UI_Switch_B1: SW_SPDT, Button_Switch_THT:SW_Slide-03_Wuerth-WS-SLTV_10x2.5x6.4_P2.54mm, symbol Switch:SW_SPDT
Connections:
- no-connect marks 64 -> 59
Other:
- note removed: "Output Stage"

Commit message: First layout attempt - large footprint
Parts:
- removed C15, C16, C3, C4, C5, C6: C, Capacitor_THT:C_Disc_D4.3mm_W1.9mm_P5.00mm, symbol Device:C
- removed D3, D4: 1N5817, Diode_THT:D_DO-41_SOD81_P10.16mm_Horizontal, symbol Diode:1N5817
- removed J3: Conn_01x04_Pin, Connector_JST:JST_PH_B4B-PH-K_1x04_P2.00mm_Vertical, symbol Connector:Conn_01x04_Pin
- removed JP1: Jumper_2_Open, Connector_PinHeader_1.00mm:PinHeader_1x02_P1.00mm_Vertical, symbol Jumper:Jumper_2_Open
- removed R10, R11, R12, R20, R6, R7, R8, R9: R, Resistor_THT:R_Axial_DIN0207_L6.3mm_D2.5mm_P7.62mm_Horizontal, symbol Device:R
- removed RV1: 500k, Potentiometer_THT:Potentiometer_Bourns_3296W_Vertical, symbol Device:R_Potentiometer_Trim
- removed RV2, RV3, RV4: 500k, Potentiometer_THT:Potentiometer_Alps_RK09Y11_Single_Horizontal, symbol Device:R_Potentiometer
- removed SW2: SW_DPDT_x2, Button_Switch_THT:SW_PUSH_E-Switch_FS5700DP_DPDT, symbol Switch:SW_DPDT_x2
- removed SW3: SW_SPDT, Button_Switch_THT:SW_Slide-03_Wuerth-WS-SLTV_10x2.5x6.4_P2.54mm, symbol Switch:SW_SPDT
- removed U1, U3: TL071, Package_DIP:DIP-8_W7.62mm, symbol Amplifier_Operational:TL071
- removed U2: LTC1044, Package_DIP:DIP-8_W7.62mm, symbol Regulator_SwitchedCapacitor:LTC1044
- removed U6: Teensy4.1, Teensy:Teensy41, symbol Teensy:Teensy4.1
- added R7: PV36W502C01B00, POT_PV36W_BRN, symbol MyComponents:PV36W502C01B00
- added U1: DM-OLED096-636, MyComponents:LED_SCREEN096, symbol MyComponents:DM-OLED096-636
- added U2: TL072, Package_DIP:DIP-8_W7.62mm, symbol Amplifier_Operational:TL072
- added U5: Teensy4.0, Teensy:Teensy40, symbol Teensy:Teensy4.0
- C1, C2: value C -> 10u
- R1, R2: value R -> 47k
- R3: value R -> 10k
- R4: value R -> 2.2k
- R5: value R -> 1k
Connections:
- net Input_Jack is gone; now on an unnamed net: J1.S
- net +3V3: now also R3.2, U1.2 (VCC_IN), U2.8 (V+), U5.16 (3V3), U5.31 (3V3)
- net GND: now also C2.1, R4.2, R5.1, U1.1 (GND), U2.4 (V-), U5.1 (GND), U5.32 (GND)
- net SCL: now also U1.3 (SCL), U5.26 (19_A5_SCL0)
- net SDA: now also U1.4 (SDA), U5.25 (18_A4_SDA0)
- net at R2.2: now also C2.2, R3.1, R4.1
- net at R5.2: now also R7.1, U2.2 (-)
- net at C1.2, R2.1: now also U2.3 (+); no longer R3.1
- net AD0 renamed A0
- net A0: now also R7.2, U2.1, U5.21 (14_A0_TX3_SPDIF_OUT)
- net FX_In: no longer names the net of C1.1, R1.1
- removed net IN_BUFFERED: C2.2, R4.2
- no-connect marks 59 -> 51
Other:
- note removed: "Power Supply"
- moved on the sheet: D1, D2, R1, R2, R3

Commit message: move toward guitar tuner
Parts:
- added J2: Conn_01x02_Socket, Connector_JST:JST_EH_B2B-EH-A_1x02_P2.50mm_Vertical, symbol Connector:Conn_01x02_Socket
Connections:
- net GND: now also J2.2 (Pin_2)
- net at U5.33 (VIN): now also J2.1 (Pin_1)
- no-connect marks 51 -> 50
Other:
- moved on the sheet: U1, U2C, U5

Commit message: Ordered Guitar Tuner
Parts:
- removed J1: AudioJack2, Connector_Audio:Jack_3.5mm_Ledino_KB3SPRS_Horizontal, symbol Connector_Audio:AudioJack2
- added J1: SJ1-3525N, MyComponents:CUI_SJ1-3525N, symbol MyComponents:SJ1-3525N
- added J3: ChargerBoard, Connector_PinHeader_2.54mm:PinHeader_1x02_P2.54mm_Vertical, symbol Connector:Conn_01x02_Socket
- added J4: BatteryConnector, Connector_PinHeader_2.54mm:PinHeader_1x02_P2.54mm_Vertical, symbol Connector:Conn_01x02_Socket
- added R6: 10k, Resistor_SMD:R_0603_1608Metric, symbol Device:R
- added SW1: SW_Push, Button_Switch_SMD:SW_SPST_B3U-3000P, symbol Switch:SW_Push
- J2: footprint Connector_JST:JST_EH_B2B-EH-A_1x02_P2.50mm_Vertical -> Connector_JST:JST_PH_B2B-PH-K_1x02_P2.00mm_Vertical
Connections:
- net +3V3: now also SW1.1
- net GND: now also J1.2, J3.2 (Pin_2), J4.2 (Pin_2), R6.1
- net at U5.13 (11_MOSI_CTX1): now also R6.2, SW1.2
- net at U5.33 (VIN): now also J3.1 (Pin_1); no longer J2.1 (Pin_1)
- net at C1.1, R1.1: now also J1.1, J1.3
- new net +BATT: J2.1 (Pin_1), J4.1 (Pin_1)
- no-connect marks 50 -> 51
Other:
- moved on the sheet: C1, C2, D1, D2, J2, R1, R2, R3, R4, R5, R7, U1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
